Commit message: 👌 IMPROVE: Simulation

File: robot_table_description/urdf/robot_table_macro.xacro (robot description, xacro)
@@ -21,4 +21,5 @@
       <visual>
         <geometry>
+          <!--<mesh filename="file://$(find robot_table_description)/meshes/robo_table.dae"/>-->
           <mesh filename="package://robot_table_description/meshes/robo_table.dae"/>
         </geometry>
@@ -27,4 +28,5 @@
       <collision>
         <geometry>
+          <!--<mesh filename="file://$(find robot_table_description)/meshes/robo_table.dae"/>-->
           <mesh filename="package://robot_table_description/meshes/robo_table.dae"/>
         </geometry>
